File: 02-hardware/wireless receiver/wireless receiver.kicad_pcb (KiCad board)
At the start: 2 copper layers, 117 parts, among them J1 Conn_HE13_1x1_5.08V, J10 Conn_HE13_1x4_2.54V, J11 Conn_HE13_1x2_2.54V, J12 Conn_HE13_1x1_5.08V, J13 Conn_HE13_1x1_5.08V, J14 Conn_HE13_1x6_2.54H, J15 Conn_HE13_1x3_2.54V, J16 Conn_HE13_1x3_2.54V, J17 Conn_HE13_1x3_2.54V, J18 Conn_HE13_1x3_2.54V, J19 Conn_HE13_1x3_2.54V, J2 Conn_HE13_1x1_5.08V, J20 Conn_HE13_1x2_2.54V, J21 Conn_HE13_1x2_2.54V, J22 Conn_HE13_1x2_2.54V, J23 Conn_HE13_1x2_2.54V, J24 Conn_HE13_1x2_2.54V, J25 Conn_HE13_1x2_2.54V, J26 Conn_HE13_1x5_2.54V, J27 Conn_HE13_1x4_2.54V, J3 Conn_HE13_1x4_2.54V, J4 Conn_HE13_1x2_2.54V, J5 Conn_HE13_1x2_2.54V, J6 Conn_HE13_1x2_2.54V, J7 Conn_HE13_1x2_2.54V, J8 Conn_HE13_1x2_2.54V, J9 Conn_HE13_1x2_2.54V, M1 nRF24L01, Q1 BC848B, Q2 BC848B, Q3 BC848B, Q4 BC848B, Q5 BC848B, U1 MAX487CSA_ESA, U10 LMV824AIYDT, U11 MCP6N11-001E_SN, U12 74HCT244, U2 TPS54332, U3 MCP1804T-5002I_O, U4 MCP1804T-3302I_O, U5 74HCT244, U6 74HCT244, U7 TCA9538, U8 REF193GSZ, U9 STM32G030_C8, Y1 Crystal_HC49CMS

Commit message: PCB base
Parts:
- removed J26: Conn_HE13_1x5_2.54V, p_Package_Misc:PinHeader_1x05_P2.54mm_Vertical
- removed J27: Conn_HE13_1x4_2.54V, p_Package_Misc:PinHeader_1x04_P2.54mm_Vertical
- J10: value Conn_HE13_1x4_2.54V -> Conn_HE13_1x1_5.08V; footprint p_Package_Misc:PinHeader_1x04_P2.54mm_Vertical -> p_Package_Misc:PinHeader_1x01_P5.08mm_Vertical
- J11: value Conn_HE13_1x2_2.54V -> Conn_HE13_1x1_5.08V; footprint p_Package_Misc:PinHeader_1x02_P2.54mm_Vertical -> p_Package_Misc:PinHeader_1x01_P5.08mm_Vertical
- J12: value Conn_HE13_1x1_5.08V -> Conn_HE13_1x6_2.54H; footprint p_Package_Misc:PinHeader_1x01_P5.08mm_Vertical -> p_Package_Misc:PinHeader_1x06_P2.54mm_Horizontal
- J13: value Conn_HE13_1x1_5.08V -> Conn_HE13_1x3_2.54V; footprint p_Package_Misc:PinHeader_1x01_P5.08mm_Vertical -> p_Package_Misc:PinHeader_1x03_P2.54mm_Vertical
- J14: value Conn_HE13_1x6_2.54H -> Conn_HE13_1x3_2.54V; footprint p_Package_Misc:PinHeader_1x06_P2.54mm_Horizontal -> p_Package_Misc:PinHeader_1x03_P2.54mm_Vertical
- J18, J19: value Conn_HE13_1x3_2.54V -> Conn_HE13_1x2_2.54V; footprint p_Package_Misc:PinHeader_1x03_P2.54mm_Vertical -> p_Package_Misc:PinHeader_1x02_P2.54mm_Vertical
- J24: value Conn_HE13_1x2_2.54V -> Conn_HE13_1x5_2.54V; footprint p_Package_Misc:PinHeader_1x02_P2.54mm_Vertical -> p_Package_Misc:PinHeader_1x05_P2.54mm_Vertical
- J25, J7: value Conn_HE13_1x2_2.54V -> Conn_HE13_1x4_2.54V; footprint p_Package_Misc:PinHeader_1x02_P2.54mm_Vertical -> p_Package_Misc:PinHeader_1x04_P2.54mm_Vertical
- J9: value Conn_HE13_1x2_2.54V -> Conn_HE13_1x6_2.54H; footprint p_Package_Misc:PinHeader_1x02_P2.54mm_Vertical -> p_Package_Misc:PinHeader_1x06_P2.54mm_Horizontal
- R1: moved to F.Cu
- R10: value 42.2k -> 100k
- R11: value 10k -> 120
- R12: value 2k -> 100k
- R13: value 0 -> 42.2k
- R14: value DNP -> 10k
- R15: value 10k -> 2k
- R16, R17, R18, R19, R20, R21, R5: value 10k -> TBD
- R2: value 120k -> TBD
- R22: value 10k -> R_0603
- R23: value 0 -> R_0603
- R24, R25: value 100k -> 10k
- R27: value 10k -> 0
- R28: value 10k -> 100k
- R29: value TBD -> 100k
- R3: value 33k -> TBD
- R30: value TBD -> 0
- R31: value TBD -> DNP
- R32, R33, R34: value TBD -> 10k
- R35, R36: value R_0603 -> 10k
- R4: value 270 -> 120k
- R6: value 100k -> 33k
- R7: value 100k -> 270
- R8: value 120 -> 10k
- U10: value LMV824AIYDT -> STM32G030_C8; footprint p_Package_SO:SO-14_3.9x8.65mm_P1.27mm -> p_Package_QFP:LQFP-48_7x7mm_P0.5mm
- U11: value MCP6N11-001E_SN -> 74HCT244; footprint p_Package_SO:SOIC-8_3.9x4.9mm_P1.27mm -> p_Package_SO:SOIC-20W_7.5x12.8mm_P1.27mm
- U5: value 74HCT244 -> LMV824AIYDT; footprint p_Package_SO:SOIC-20W_7.5x12.8mm_P1.27mm -> p_Package_SO:SO-14_3.9x8.65mm_P1.27mm
- U6: value 74HCT244 -> MCP6N11-001E_SN; footprint p_Package_SO:SOIC-20W_7.5x12.8mm_P1.27mm -> p_Package_SO:SOIC-8_3.9x4.9mm_P1.27mm
- U7: value TCA9538 -> 74HCT244; footprint p_Package_SO:SSOP-16_5.3x6.2mm_P0.65mm -> p_Package_SO:SOIC-20W_7.5x12.8mm_P1.27mm
- U8: value REF193GSZ -> TCA9538; footprint p_Package_SO:SOIC-8_3.9x4.9mm_P1.27mm -> p_Package_SO:SSOP-16_5.3x6.2mm_P0.65mm
- U9: value STM32G030_C8 -> REF193GSZ; footprint p_Package_QFP:LQFP-48_7x7mm_P0.5mm -> p_Package_SO:SOIC-8_3.9x4.9mm_P1.27mm
- moved R34 205.2 mm to (13.3, 82.2)
- moved R32 197.1 mm to (27.8, 80.8)
- moved U12 192.7 mm to (17.6, 67.8)
- moved R35 190.9 mm to (17.7, 82.2)
- moved R33 190.4 mm to (23.4, 80.8)
- moved C26 190.1 mm to (39.2, 74.0)
- moved R31 181.6 mm to (32.3, 76.3)
- moved U11 179.0 mm to (30.5, 67.8)
- moved R36 177.4 mm to (43.6, 66.5)
- moved C25 167.1 mm to (48.7, 64.4)
- moved J24 165.3 mm to (26.9, 35.1)
- moved J21 160.4 mm to (40.8, 50.0)
- moved R23 158.4 mm to (103.8, 66.9)
- moved J7 155.3 mm to (31.5, 35.6)
- moved R22 155.3 mm to (95.4, 70.6)
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Connections:
- C11 pad 1: +3V3 -> +3.3V
- C16 pad 1: /output_stage/VCC_74HCT244 -> +3.3V
- C17 pad 1: /output_stage/VCC_74HCT244 -> +3.3V
- C18 pad 1: +3V3 -> +3.3V
- C19 pad 1: +3V3 -> +3.3V
- C20 pad 1: +3V3 -> +3.3V
- C21 pad 1: +3V3 -> +3.3V
- C25 pad 1: +3V3 -> /output_stage/VCC_74HCT244
- C26 pad 1: +3V3 -> GND
- C26 pad 2: GND -> /output_stage/VCC_74HCT244
- J10 pad 1: /input_stage/INPUT1 -> GND
- J11 pad 1: /input_stage/LOOPBACK1 -> +BATT
- J12 pad 1: GND -> +3.3V
- J13 pad 1: +BATT -> /output_stage/SERVO1_CMD
- J14 pad 1: +3V3 -> /output_stage/SERVO2_CMD
- J14 pad 2: /SWDIO -> +5VP
- J14 pad 3: /SWCLK -> GND
- J15 pad 1: /output_stage/SERVO1_CMD -> /output_stage/SERVO3_CMD
- J16 pad 1: /output_stage/SERVO2_CMD -> /output_stage/SERVO4_CMD
- J17 pad 1: /output_stage/SERVO3_CMD -> /output_stage/SERVO5_CMD
- J18 pad 1: /output_stage/SERVO4_CMD -> /output_stage/OUTPUT1_LVL
- J18 pad 2: +5VP -> GND
- J19 pad 1: /output_stage/SERVO5_CMD -> /output_stage/OUTPUT2_LVL
- J19 pad 2: +5VP -> GND
- J20 pad 1: /output_stage/OUTPUT1_LVL -> /output_stage/OUTPUT3_LVL
- J21 pad 1: /output_stage/OUTPUT2_LVL -> /output_stage/OUTPUT4_LVL
- J22 pad 1: /output_stage/OUTPUT3_LVL -> /output_stage/OUTPUT5_LVL
- J23 pad 1: /output_stage/OUTPUT4_LVL -> /output_stage/OUTPUT6_LVL
- J24 pad 1: /output_stage/OUTPUT5_LVL -> /output_stage/OUTPUT7_ODRAIN
- J24 pad 2: GND -> /output_stage/OUTPUT8_ODRAIN
- J25 pad 1: /output_stage/OUTPUT6_LVL -> +5VP
- J25 pad 2: GND -> Net-(J25-Pad2)
- J3 pad 1: +3V3 -> +3.3V
- J4 pad 1: /MCU/TEMP1 -> /MCU/TEMP3
- J6 pad 1: /MCU/TEMP3 -> /MCU/TEMP1
- J7 pad 1: /analog_input_stage/V_MONITOR1 -> /input_stage/INPUT1
- J7 pad 2: GND -> /input_stage/INPUT2
- J8 pad 1: /analog_input_stage/V_MONITOR2 -> /input_stage/LOOPBACK1
- J8 pad 2: GND -> /input_stage/LOOPBACK2
- J9 pad 1: /analog_input_stage/V_MONITOR3 -> /analog_input_stage/V_MONITOR1
- M1 pad 2: +3V3 -> +3.3V
- M1 pad 4: /~CS_NRF24L01~ -> /~{CS_NRF24L01}
- R10 pad 1: Net-(C12-Pad1) -> /MCU/TX_EN
- R10 pad 2: Net-(C13-Pad1) -> GND
- R11 pad 1: +5VP -> Net-(J25-Pad2)
- R11 pad 2: Net-(R11-Pad2) -> Net-(J25-Pad3)
- R12 pad 1: Net-(R11-Pad2) -> /MCU/EN_5V_PWR
- R13 pad 1: /output_stage/VCC_74HCT244 -> Net-(C12-Pad1)
- R13 pad 2: +5V -> Net-(C13-Pad1)
- R14 pad 1: /output_stage/VCC_74HCT244 -> +5VP
- R14 pad 2: +3V3 -> Net-(R14-Pad2)
- R15 pad 1: Net-(Q1-Pad2) -> Net-(R14-Pad2)
- R15 pad 2: Net-(R15-Pad2) -> GND
- R16 pad 1: Net-(Q2-Pad2) -> /MCU/ADC_MONITOR1
- R17 pad 1: Net-(Q3-Pad2) -> /MCU/ADC_MONITOR2
- R18 pad 1: Net-(Q4-Pad2) -> /MCU/ADC_MONITOR3
- R19 pad 1: Net-(Q5-Pad2) -> GND
- R19 pad 2: Net-(R19-Pad2) -> /MCU/ADC_MONITOR1
- R2 pad 1: /MCU/VBATT_MONITOR -> +3.3V
- R2 pad 2: +BATT -> /MCU/TEMP3
- R20 pad 1: +3V3 -> GND
- R20 pad 2: /I2C_SCL -> /MCU/ADC_MONITOR2
- R21 pad 1: +3V3 -> GND
- R21 pad 2: /I2C_SDA -> /MCU/ADC_MONITOR3
- R22 pad 1: +3V3 -> /MCU/ADC_CURRENT_MEAS
- R23 pad 1: Net-(C24-Pad2) -> Net-(R22-Pad2)
- R23 pad 2: Net-(R23-Pad2) -> GND
- R24 pad 1: GND -> +3.3V
- R24 pad 2: Net-(R24-Pad2) -> /I2C_SCL
- R25 pad 1: +5VP -> +3.3V
- R25 pad 2: Net-(R24-Pad2) -> /I2C_SDA
- R26 pad 1: +3V3 -> +3.3V
- R26 pad 2: /MCU/TEMP1 -> Net-(R26-Pad2)
- R27 pad 1: +3V3 -> Net-(C24-Pad2)
- R27 pad 2: /MCU/TEMP2 -> Net-(R27-Pad2)
- R28 pad 1: +3V3 -> GND
- R28 pad 2: /MCU/TEMP3 -> Net-(R28-Pad2)
- R29 pad 1: /MCU/ADC_MONITOR1 -> +5VP
- R29 pad 2: Net-(R29-Pad2) -> Net-(R28-Pad2)
- R3 pad 1: GND -> +3.3V
- R3 pad 2: /MCU/VBATT_MONITOR -> /MCU/TEMP2
- R30 pad 1: /MCU/ADC_MONITOR2 -> /output_stage/VCC_74HCT244
- R30 pad 2: Net-(R30-Pad2) -> +5V
- R31 pad 1: /MCU/ADC_MONITOR3 -> /output_stage/VCC_74HCT244
- R31 pad 2: Net-(R31-Pad2) -> +3.3V
- R32 pad 1: GND -> Net-(Q1-Pad2)
- R32 pad 2: /MCU/ADC_MONITOR1 -> Net-(R32-Pad2)
- R33 pad 1: GND -> Net-(Q2-Pad2)
- R33 pad 2: /MCU/ADC_MONITOR2 -> Net-(R33-Pad2)
- R34 pad 1: GND -> Net-(Q3-Pad2)
- R34 pad 2: /MCU/ADC_MONITOR3 -> Net-(R34-Pad2)
- R35 pad 1: /MCU/ADC_CURRENT_MEAS -> Net-(Q4-Pad2)
- R36 pad 1: Net-(R35-Pad2) -> Net-(Q5-Pad2)
- R36 pad 2: GND -> Net-(R36-Pad2)
- R4 pad 1: Net-(D2-Pad2) -> /MCU/VBATT_MONITOR
- R4 pad 2: +3V3 -> +BATT
- R5 pad 1: +3V3 -> +3.3V
- R5 pad 2: /~RESET~ -> /MCU/TEMP1
- R6 pad 2: /CE_NRF24L01 -> /MCU/VBATT_MONITOR
- R7 pad 1: /MCU/TX_EN -> Net-(D2-Pad2)
- R7 pad 2: GND -> +3.3V
- R8 pad 1: Net-(J27-Pad2) -> +3.3V
- R8 pad 2: Net-(J27-Pad3) -> /~{RESET}
- R9 pad 1: /MCU/EN_5V_PWR -> GND
- R9 pad 2: GND -> /CE_NRF24L01
- U1 pad 2: /MCU/~RX_EN~ -> /MCU/~{RX_EN}
- U1 pad 6: Net-(J27-Pad2) -> Net-(J25-Pad2)
- U1 pad 7: Net-(J27-Pad3) -> Net-(J25-Pad3)
- U10 pad 1: Net-(R29-Pad2) -> /MCU/INPUT3
- U10 pad 10: /analog_input_stage/V_MONITOR3 -> /~{RESET}
- U10 pad 11: +3V3 -> /MCU/VBATT_MONITOR
- U10 pad 12: GND -> /MCU/~{EN_VREF}
- U10 pad 13: GND -> /IRQ_NRF24L01
- U10 pad 14: Net-(U10-Pad14) -> /MCU/OUTPUT1
- U10 pad 2: /analog_input_stage/V_MONITOR1 -> /MCU/INPUT4
- U10 pad 3: Net-(R29-Pad2) -> /MCU/OUTPUT2
- U10 pad 4: GND -> +3.3V
- U10 pad 5: /analog_input_stage/V_MONITOR2 -> /MCU/VREF
- U10 pad 6: Net-(R30-Pad2) -> +3.3V
- U10 pad 7: Net-(R30-Pad2) -> GND
- U10 pad 8: Net-(R31-Pad2) -> Net-(C23-Pad2)
- U10 pad 9: Net-(R31-Pad2) -> Net-(R27-Pad2)
- U11 pad 1: Net-(R35-Pad2) -> GND
- U11 pad 2: /BAT_SENSE- -> /MCU/PWM1
- U11 pad 3: /BAT_SENSE+ -> /output_stage/SERVO5_CMD
- U11 pad 4: GND -> /MCU/PWM2
- U11 pad 5: GND -> /output_stage/OUTPUT1_LVL
- U11 pad 6: /MCU/ADC_CURRENT_MEAS -> /MCU/PWM3
- U11 pad 7: +3V3 -> /output_stage/OUTPUT2_LVL
- U11 pad 8: +3V3 -> /MCU/PWM4
- U12 pad 11: GND -> /MCU/OUTPUT11
- U12 pad 12: /input_stage/IN4 -> Net-(R32-Pad2)
- U12 pad 13: GND -> /MCU/OUTPUT10
- U12 pad 14: /input_stage/IN3 -> /output_stage/OUTPUT6_LVL
- U12 pad 15: /input_stage/LOOPBACK2 -> /MCU/OUTPUT9
- U12 pad 16: /input_stage/IN2 -> /output_stage/OUTPUT5_LVL
- U12 pad 17: /input_stage/LOOPBACK1 -> /MCU/OUTPUT8
- U12 pad 18: /input_stage/IN1 -> /output_stage/OUTPUT4_LVL
- U12 pad 2: /input_stage/INPUT1 -> /MCU/OUTPUT4
- U12 pad 20: +3V3 -> /output_stage/VCC_74HCT244
- U12 pad 3: /MCU/LOOPBACK1 -> Net-(R33-Pad2)
- U12 pad 4: /input_stage/INPUT2 -> /MCU/OUTPUT5
- U12 pad 5: /MCU/LOOPBACK2 -> Net-(R34-Pad2)
- U12 pad 6: /input_stage/INPUT3 -> /MCU/OUTPUT6
- U12 pad 7: Net-(U12-Pad7) -> Net-(R35-Pad2)
- U12 pad 8: /input_stage/INPUT4 -> /MCU/OUTPUT7
- U12 pad 9: Net-(U12-Pad9) -> Net-(R36-Pad2)
- U2 pad 5: Net-(R11-Pad2) -> Net-(R14-Pad2)
- U3 pad 3: Net-(U3-Pad3) -> unconnected-(U3-Pad3)
- U4 pad 3: Net-(U4-Pad3) -> unconnected-(U4-Pad3)
- U4 pad 5: +3V3 -> +3.3V
- U5 pad 1: GND -> Net-(R16-Pad2)
- U5 pad 10: GND -> /analog_input_stage/V_MONITOR3
- U5 pad 11: /MCU/OUTPUT3 -> GND
- U5 pad 12: /output_stage/SERVO4_CMD -> GND
- U5 pad 13: /MCU/OUTPUT2 -> GND
- U5 pad 14: /output_stage/SERVO3_CMD -> unconnected-(U5-Pad14)
- U5 pad 2: /MCU/PWM1 -> Net-(R16-Pad2)
- U5 pad 3: /output_stage/SERVO5_CMD -> /analog_input_stage/V_MONITOR1
- U5 pad 4: /MCU/PWM2 -> +3.3V
- U5 pad 5: /output_stage/OUTPUT1_LVL -> /analog_input_stage/V_MONITOR2
- U5 pad 6: /MCU/PWM3 -> Net-(R17-Pad2)
- U5 pad 7: /output_stage/OUTPUT2_LVL -> Net-(R17-Pad2)
- U5 pad 8: /MCU/PWM4 -> Net-(R18-Pad2)
- U5 pad 9: /output_stage/OUTPUT3_LVL -> Net-(R18-Pad2)
- U6 pad 1: GND -> Net-(R22-Pad2)
- U6 pad 2: /MCU/OUTPUT4 -> /BAT_SENSE-
- U6 pad 3: Net-(R16-Pad2) -> /BAT_SENSE+
- U6 pad 4: /MCU/OUTPUT5 -> GND
- U6 pad 5: Net-(R17-Pad2) -> GND
- U6 pad 6: /MCU/OUTPUT6 -> /MCU/ADC_CURRENT_MEAS
- U6 pad 7: Net-(R18-Pad2) -> +3.3V
- U6 pad 8: /MCU/OUTPUT7 -> +3.3V
- U7 pad 10: /MCU/~RX_EN~ -> GND
- U7 pad 11: /CE_NRF24L01 -> GND
- U7 pad 12: /MCU/EN_5V_PWR -> /MCU/INPUT4
- U7 pad 13: /MCU/~INT~ -> GND
- U7 pad 14: /I2C_SCL -> /MCU/INPUT3
- U7 pad 15: /I2C_SDA -> /input_stage/LOOPBACK2
- U7 pad 16: +3V3 -> /MCU/INPUT2
- U7 pad 2: GND -> /input_stage/INPUT1
- U7 pad 3: Net-(R22-Pad2) -> /MCU/LOOPBACK1
- U7 pad 4: /MCU/OUTPUT8 -> /input_stage/INPUT2
- U7 pad 5: /MCU/OUTPUT9 -> /MCU/LOOPBACK2
- U7 pad 6: /MCU/OUTPUT10 -> /input_stage/INPUT3
- U7 pad 7: /MCU/OUTPUT11 -> unconnected-(U7-Pad7)
- U7 pad 8: GND -> /input_stage/INPUT4
- U7 pad 9: /MCU/TX_EN -> unconnected-(U7-Pad9)
- U8 pad 1: Net-(U8-Pad1) -> GND
- U8 pad 2: +3V3 -> GND
- U8 pad 3: /MCU/~EN_VREF~ -> Net-(R26-Pad2)
- U8 pad 4: GND -> /MCU/OUTPUT8
- U8 pad 5: Net-(U8-Pad5) -> /MCU/OUTPUT9
- U8 pad 6: /MCU/VREF -> /MCU/OUTPUT10
- U8 pad 7: Net-(U8-Pad7) -> /MCU/OUTPUT11
- U8 pad 8: Net-(U8-Pad8) -> GND
- U9 pad 1: /input_stage/IN3 -> unconnected-(U9-Pad1)
- U9 pad 2: /input_stage/IN4 -> +3.3V
- U9 pad 3: /MCU/OUTPUT2 -> /MCU/~{EN_VREF}
- U9 pad 4: +3V3 -> GND
- U9 pad 5: /MCU/VREF -> unconnected-(U9-Pad5)
- U9 pad 6: +3V3 -> /MCU/VREF
- U9 pad 7: GND -> unconnected-(U9-Pad7)
- U9 pad 8: Net-(C23-Pad2) -> unconnected-(U9-Pad8)
Other:
- net class Default removed
