File: 02-hardware/wireless receiver/MCU.kicad_sch (KiCad schematic)
At the start: 17 parts, among them U10 STM32G030_C8, U8 TCA9538, U9 REF193GSZ, Y1 Crystal_HC49CMS

Commit message: wip
Connections:
- net LOOPBACK1 is gone; now on net OUTPUT5: U10.39 (PD1)
- net LOOPBACK2 is gone; now on net OUTPUT6: U10.40 (PD2)
- net ADC_CURRENT_MEAS: now also U10.16 (PA5); no longer U10.24 (PB12)
- net INPUT3: now also U10.12 (PA1); no longer U10.1 (PC13)
- net INPUT4: now also U10.3 (PC15); no longer U10.2 (PC14)
- net IRQ_NRF24L01: now also U10.14 (PA3); no longer U10.13 (PA2)
- net OUTPUT1: now also U10.15 (PA4); no longer U10.14 (PA3)
- net OUTPUT2: now also U10.2 (PC14); no longer U10.3 (PC15)
- net OUTPUT5: no longer U10.33 (PA11)
- net OUTPUT6: no longer U10.34 (PA12)
- net OUTPUT7: now also U10.41 (PD3); no longer U10.37 (PA15)
- net TEMP1: now also U10.24 (PB12); no longer U10.16 (PA5)
- net ~{CS_NRF24L01}: now also U10.13 (PA2); no longer U10.15 (PA4)
- net ~{EN_VREF}: now also U10.1 (PC13); no longer U10.12 (PA1)
- net ~{INT}: now also U10.37 (PA15); no longer U10.41 (PD3)
- new net GPIO1: U10.33 (PA11)
- new net GPIO2: U10.34 (PA12)
