File: 02-hardware/wireless receiver/input_stage.kicad_sch (KiCad schematic)
At the start: 2 parts, among them U7 74HCT244

Commit message: wip
Connections:
- net LOOPBACK1 is gone; now on net GND: U7.17 (2A0)
- net LOOPBACK2 is gone; now on net GND: U7.15 (2A1)
- net LP1: no longer names the net of U7.3 (2Y0)
- net LP2: no longer names the net of U7.5 (2Y1)
- no-connect marks 2 -> 4
Changed lines of the file:
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@@
   (junction (at 123.19 109.22) (diameter 0) (color 0 0 0 0)
   )
+  (junction (at 123.19 96.52) (diameter 0) (color 0 0 0 0)
+  )
+  (junction (at 123.19 99.06) (diameter 0) (color 0 0 0 0)
+  )
   (junction (at 123.19 106.68) (diameter 0) (color 0 0 0 0)
   )
+  (no_connect (at 151.13 96.52))
+  (no_connect (at 151.13 93.98))
   (no_connect (at 151.13 99.06))
   (no_connect (at 151.13 101.6))
@@
     (stroke (width 0) (type default) (color 0 0 0 0))
   )
-  (wire (pts (xy 82.55 93.98) (xy 125.73 93.98))
-    (stroke (width 0) (type default) (color 0 0 0 0))
-  )
   (wire (pts (xy 85.09 63.5) (xy 85.09 60.96))
     (stroke (width 0) (type default) (color 0 0 0 0))
@@
     (stroke (width 0) (type default) (color 0 0 0 0))
   )
+  (wire (pts (xy 125.73 93.98) (xy 123.19 93.98))
+    (stroke (width 0) (type default) (color 0 0 0 0))
+  )
   (wire (pts (xy 123.19 110.49) (xy 123.19 109.22))
     (stroke (width 0) (type default) (color 0 0 0 0))
@@
     (stroke (width 0) (type default) (color 0 0 0 0))
   )
-  (wire (pts (xy 82.55 96.52) (xy 125.73 96.52))
+  (wire (pts (xy 123.19 93.98) (xy 123.19 96.52))
     (stroke (width 0) (type default) (color 0 0 0 0))
   )
@@
     (stroke (width 0) (type default) (color 0 0 0 0))
   )
-  (wire (pts (xy 231.14 96.52) (xy 151.13 96.52))
-    (stroke (width 0) (type default) (color 0 0 0 0))
-  )
   (wire (pts (xy 231.14 88.9) (xy 151.13 88.9))
     (stroke (width 0) (type default) (color 0 0 0 0))
   )
-  (wire (pts (xy 151.13 93.98) (xy 231.14 93.98))
+  (wire (pts (xy 123.19 96.52) (xy 123.19 99.06))
     (stroke (width 0) (type default) (color 0 0 0 0))
   )
@@
     (stroke (width 0) (type default) (color 0 0 0 0))
   )
-  (hierarchical_label "LOOPBACK1" (shape input) (at 82.55 93.98 180)
-    (effects (font (size 1.27 1.27)) (justify right))
-  )
-  (hierarchical_label "LP2" (shape output) (at 231.14 96.52 0)
-    (effects (font (size 1.27 1.27)) (justify left))
+  (wire (pts (xy 125.73 96.52) (xy 123.19 96.52))
+    (stroke (width 0) (type default) (color 0 0 0 0))
   )
   (hierarchical_label "GND" (shape passive) (at 82.55 121.92 180)
@@
     (effects (font (size 1.27 1.27)) (justify left))
   )
-  (hierarchical_label "LOOPBACK2" (shape input) (at 82.55 96.52 180)
-    (effects (font (size 1.27 1.27)) (justify right))
-  )
   (hierarchical_label "+3.3V" (shape passive) (at 82.55 63.5 180)
     (effects (font (size 1.27 1.27)) (justify right))
@@
   (hierarchical_label "INPUT3" (shape input) (at 82.55 86.36 180)
     (effects (font (size 1.27 1.27)) (justify right))
-  )
-  (hierarchical_label "LP1" (shape output) (at 231.14 93.98 0)
-    (effects (font (size 1.27 1.27)) (justify left))
   )
   (hierarchical_label "IN2" (shape output) (at 231.14 83.82 0)
@@
   (symbol (lib_id "power:GND") (at 85.09 123.19 0) (unit 1)
     (in_bom yes) (on_board yes)
-    (property "Reference" "#PWR066" (id 0) (at 85.09 129.54 0)
+    (property "Reference" "#PWR067" (id 0) (at 85.09 129.54 0)
       (effects (font (size 1.27 1.27)) hide)
     )
@@
   (symbol (lib_id "power:GND") (at 123.19 110.49 0) (unit 1)
     (in_bom yes) (on_board yes)
-    (property "Reference" "#PWR067" (id 0) (at 123.19 116.84 0)
+    (property "Reference" "#PWR068" (id 0) (at 123.19 116.84 0)
       (effects (font (size 1.27 1.27)) hide)
     )
@@
   (symbol (lib_id "power:GND") (at 153.67 110.49 0) (unit 1)
     (in_bom yes) (on_board yes)
-    (property "Reference" "#PWR068" (id 0) (at 153.67 116.84 0)
+    (property "Reference" "#PWR069" (id 0) (at 153.67 116.84 0)
       (effects (font (size 1.27 1.27)) hide)
     )
@@
   (symbol (lib_id "power:GND") (at 158.75 74.93 0) (unit 1)
     (in_bom yes) (on_board yes)
-    (property "Reference" "#PWR070" (id 0) (at 158.75 81.28 0)
+    (property "Reference" "#PWR071" (id 0) (at 158.75 81.28 0)
       (effects (font (size 1.27 1.27)) hide)
     )
@@
   (symbol (lib_id "power:+3.3V") (at 85.09 60.96 0) (unit 1)
     (in_bom yes) (on_board yes)
-    (property "Reference" "#PWR065" (id 0) (at 85.09 64.77 0)
+    (property "Reference" "#PWR066" (id 0) (at 85.09 64.77 0)
       (effects (font (size 1.27 1.27)) hide)
     )
@@
   (symbol (lib_id "power:+3.3V") (at 158.75 63.5 0) (unit 1)
     (in_bom yes) (on_board yes)
-    (property "Reference" "#PWR069" (id 0) (at 158.75 67.31 0)
-      (effects (font (size 1.27 1.27)) hide)
-    )
+    (property "Reference" "#PWR070" (id 0) (at 158.75 67.31 0)
+      (effects (font (size 1.27 1.27)) hide)
+    )
