File: 02-hardware/wireless receiver/output_stage.kicad_sch (KiCad schematic)
At the start: 21 parts, among them Q1 BC848B, Q2 BC848B, Q3 BC848B, Q4 BC848B, Q5 BC848B, U11 74HCT244, U12 74HCT244

Commit message: wip
Connections:
- net OUTPUT1: now also U11.11 (2A3); no longer U11.15 (2A1)
- net OUTPUT1_LVL: now also U11.9 (2Y3); no longer U11.5 (2Y1)
- net OUTPUT2: now also U11.8 (1A3); no longer U11.13 (2A2)
- net OUTPUT2_LVL: now also U11.12 (1Y3); no longer U11.7 (2Y2)
- net OUTPUT3: now also U11.4 (1A1); no longer U11.11 (2A3)
- net OUTPUT3_LVL: now also U11.16 (1Y1); no longer U11.9 (2Y3)
- net PWM2: now also U11.17 (2A0); no longer U11.4 (1A1)
- net PWM4: now also U11.13 (2A2); no longer U11.8 (1A3)
- net PWM5: now also U11.15 (2A1); no longer U11.17 (2A0)
- net SERVO2_CMD: now also U11.3 (2Y0); no longer U11.16 (1Y1)
- net SERVO4_CMD: now also U11.7 (2Y2); no longer U11.12 (1Y3)
- net SERVO5_CMD: now also U11.5 (2Y1); no longer U11.3 (2Y0)
Changed lines of the file:
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@@
     (effects (font (size 1.27 1.27)) (justify right))
   )
-  (hierarchical_label "OUTPUT3_LVL" (shape output) (at 195.58 57.15 0)
+  (hierarchical_label "OUTPUT3_LVL" (shape output) (at 195.58 39.37 0)
     (effects (font (size 1.27 1.27)) (justify left))
   )
@@
     (effects (font (size 1.27 1.27)) (justify left))
   )
-  (hierarchical_label "OUTPUT2" (shape input) (at 38.1 54.61 180)
+  (hierarchical_label "OUTPUT2" (shape input) (at 38.1 44.45 180)
     (effects (font (size 1.27 1.27)) (justify right))
   )
@@
     (effects (font (size 1.27 1.27)) (justify right))
   )
-  (hierarchical_label "SERVO2_CMD" (shape output) (at 195.58 39.37 0)
-    (effects (font (size 1.27 1.27)) (justify left))
-  )
-  (hierarchical_label "PWM5" (shape input) (at 38.1 49.53 180)
-    (effects (font (size 1.27 1.27)) (justify right))
-  )
-  (hierarchical_label "SERVO5_CMD" (shape output) (at 195.58 49.53 0)
+  (hierarchical_label "SERVO2_CMD" (shape output) (at 195.58 49.53 0)
+    (effects (font (size 1.27 1.27)) (justify left))
+  )
+  (hierarchical_label "PWM5" (shape input) (at 38.1 52.07 180)
+    (effects (font (size 1.27 1.27)) (justify right))
+  )
+  (hierarchical_label "SERVO5_CMD" (shape output) (at 195.58 52.07 0)
     (effects (font (size 1.27 1.27)) (justify left))
   )
@@
     (effects (font (size 1.27 1.27)) (justify right))
   )
-  (hierarchical_label "OUTPUT2_LVL" (shape output) (at 195.58 54.61 0)
+  (hierarchical_label "OUTPUT2_LVL" (shape output) (at 195.58 44.45 0)
     (effects (font (size 1.27 1.27)) (justify left))
   )
@@
     (effects (font (size 1.27 1.27)) (justify left))
   )
-  (hierarchical_label "PWM4" (shape input) (at 38.1 44.45 180)
-    (effects (font (size 1.27 1.27)) (justify right))
-  )
-  (hierarchical_label "OUTPUT3" (shape input) (at 38.1 57.15 180)
-    (effects (font (size 1.27 1.27)) (justify right))
-  )
-  (hierarchical_label "OUTPUT1_LVL" (shape output) (at 195.58 52.07 0)
+  (hierarchical_label "PWM4" (shape input) (at 38.1 54.61 180)
+    (effects (font (size 1.27 1.27)) (justify right))
+  )
+  (hierarchical_label "OUTPUT3" (shape input) (at 38.1 39.37 180)
+    (effects (font (size 1.27 1.27)) (justify right))
+  )
+  (hierarchical_label "OUTPUT1_LVL" (shape output) (at 195.58 57.15 0)
     (effects (font (size 1.27 1.27)) (justify left))
   )
@@
     (effects (font (size 1.27 1.27)) (justify right))
   )
-  (hierarchical_label "PWM2" (shape input) (at 38.1 39.37 180)
+  (hierarchical_label "PWM2" (shape input) (at 38.1 49.53 180)
     (effects (font (size 1.27 1.27)) (justify right))
   )
@@
     (effects (font (size 1.27 1.27)) (justify right))
   )
-  (hierarchical_label "OUTPUT1" (shape input) (at 38.1 52.07 180)
-    (effects (font (size 1.27 1.27)) (justify right))
-  )
-  (hierarchical_label "SERVO4_CMD" (shape output) (at 195.58 44.45 0)
+  (hierarchical_label "OUTPUT1" (shape input) (at 38.1 57.15 180)
+    (effects (font (size 1.27 1.27)) (justify right))
+  )
+  (hierarchical_label "SERVO4_CMD" (shape output) (at 195.58 54.61 0)
     (effects (font (size 1.27 1.27)) (justify left))
   )
@@
   (symbol (lib_id "power:GND") (at 81.28 66.04 0) (unit 1)
     (in_bom yes) (on_board yes)
-    (property "Reference" "#PWR092" (id 0) (at 81.28 72.39 0)
+    (property "Reference" "#PWR093" (id 0) (at 81.28 72.39 0)
       (effects (font (size 1.27 1.27)) hide)
     )
@@
   (symbol (lib_id "power:GND") (at 53.34 66.04 0) (unit 1)
     (in_bom yes) (on_board yes)
-    (property "Reference" "#PWR090" (id 0) (at 53.34 72.39 0)
+    (property "Reference" "#PWR091" (id 0) (at 53.34 72.39 0)
       (effects (font (size 1.27 1.27)) hide)
     )
@@
   (symbol (lib_id "power:GND") (at 81.28 142.24 0) (unit 1)
     (in_bom yes) (on_board yes)
-    (property "Reference" "#PWR093" (id 0) (at 81.28 148.59 0)
+    (property "Reference" "#PWR094" (id 0) (at 81.28 148.59 0)
       (effects (font (size 1.27 1.27)) hide)
     )
@@
   (symbol (lib_id "power:GND") (at 53.34 142.24 0) (unit 1)
     (in_bom yes) (on_board yes)
-    (property "Reference" "#PWR091" (id 0) (at 53.34 148.59 0)
+    (property "Reference" "#PWR092" (id 0) (at 53.34 148.59 0)
       (effects (font (size 1.27 1.27)) hide)
     )
@@
   (symbol (lib_id "power:PWR_FLAG") (at 52.07 161.29 0) (unit 1)
     (in_bom yes) (on_board yes)
-    (property "Reference" "#FLG03" (id 0) (at 52.07 159.385 0)
+    (property "Reference" "#FLG04" (id 0) (at 52.07 159.385 0)
       (effects (font (size 1.27 1.27)) hide)
     )
@@
   (symbol (lib_id "power:GND") (at 156.21 93.98 0) (unit 1)
     (in_bom yes) (on_board yes)
-    (property "Reference" "#PWR096" (id 0) (at 156.21 100.33 0)
+    (property "Reference" "#PWR097" (id 0) (at 156.21 100.33 0)
       (effects (font (size 1.27 1.27)) hide)
     )
@@
   (symbol (lib_id "power:GND") (at 156.21 114.3 0) (unit 1)
     (in_bom yes) (on_board yes)
-    (property "Reference" "#PWR097" (id 0) (at 156.21 120.65 0)
+    (property "Reference" "#PWR098" (id 0) (at 156.21 120.65 0)
       (effects (font (size 1.27 1.27)) hide)
     )
@@
   (symbol (lib_id "power:GND") (at 156.21 134.62 0) (unit 1)
     (in_bom yes) (on_board yes)
-    (property "Reference" "#PWR098" (id 0) (at 156.21 140.97 0)
+    (property "Reference" "#PWR099" (id 0) (at 156.21 140.97 0)
       (effects (font (size 1.27 1.27)) hide)
     )
@@
   (symbol (lib_id "power:GND") (at 156.21 154.94 0) (unit 1)
     (in_bom yes) (on_board yes)
-    (property "Reference" "#PWR099" (id 0) (at 156.21 161.29 0)
+    (property "Reference" "#PWR0100" (id 0) (at 156.21 161.29 0)
       (effects (font (size 1.27 1.27)) hide)
     )
@@
   (symbol (lib_id "power:GND") (at 156.21 175.26 0) (unit 1)
     (in_bom yes) (on_board yes)
-    (property "Reference" "#PWR0100" (id 0) (at 156.21 181.61 0)
+    (property "Reference" "#PWR0101" (id 0) (at 156.21 181.61 0)
       (effects (font (size 1.27 1.27)) hide)
     )
@@
   (symbol (lib_id "power:GND") (at 171.45 93.98 0) (unit 1)
     (in_bom yes) (on_board yes)
-    (property "Reference" "#PWR0101" (id 0) (at 171.45 100.33 0)
+    (property "Reference" "#PWR0102" (id 0) (at 171.45 100.33 0)
       (effects (font (size 1.27 1.27)) hide)
     )
@@
   (symbol (lib_id "power:GND") (at 171.45 114.3 0) (unit 1)
     (in_bom yes) (on_board yes)
-    (property "Reference" "#PWR0102" (id 0) (at 171.45 120.65 0)
+    (property "Reference" "#PWR0103" (id 0) (at 171.45 120.65 0)
       (effects (font (size 1.27 1.27)) hide)
     )
@@
   (symbol (lib_id "power:GND") (at 171.45 134.62 0) (unit 1)
     (in_bom yes) (on_board yes)
-    (property "Reference" "#PWR0103" (id 0) (at 171.45 140.97 0)
+    (property "Reference" "#PWR0104" (id 0) (at 171.45 140.97 0)
       (effects (font (size 1.27 1.27)) hide)
     )
@@
   (symbol (lib_id "power:GND") (at 171.45 154.94 0) (unit 1)
     (in_bom yes) (on_board yes)
-    (property "Reference" "#PWR0104" (id 0) (at 171.45 161.29 0)
+    (property "Reference" "#PWR0105" (id 0) (at 171.45 161.29 0)
       (effects (font (size 1.27 1.27)) hide)
     )
@@
   (symbol (lib_id "power:GND") (at 171.45 175.26 0) (unit 1)
     (in_bom yes) (on_board yes)
-    (property "Reference" "#PWR0105" (id 0) (at 171.45 181.61 0)
+    (property "Reference" "#PWR0106" (id 0) (at 171.45 181.61 0)
       (effects (font (size 1.27 1.27)) hide)
     )
@@
   (symbol (lib_id "power:GND") (at 39.37 187.96 0) (unit 1)
     (in_bom yes) (on_board yes)
-    (property "Reference" "#PWR089" (id 0) (at 39.37 194.31 0)
+    (property "Reference" "#PWR090" (id 0) (at 39.37 194.31 0)
       (effects (font (size 1.27 1.27)) hide)
     )
@@
   (symbol (lib_id "power:GND") (at 85.09 30.48 0) (unit 1)
     (in_bom yes) (on_board yes)
-    (property "Reference" "#PWR094" (id 0) (at 85.09 36.83 0)
+    (property "Reference" "#PWR095" (id 0) (at 85.09 36.83 0)
       (effects (font (size 1.27 1.27)) hide)
     )
@@
   (symbol (lib_id "power:GND") (at 85.09 106.68 0) (unit 1)
     (in_bom yes) (on_board yes) (fields_autoplaced)
-    (property "Reference" "#PWR0110" (id 0) (at 85.09 113.03 0)
-      (effects (font (size 1.27 1.27)) hide)
-    )
+    (property "Reference" "#PWR096" (id 0) (at 85.09 113.03 0)
+      (effects (font (size 1.27 1.27)) hide)
+    )
