File: 02-hardware/wireless receiver/wireless receiver.kicad_sch (KiCad schematic)
At the start: 41 parts, among them J1 Conn_HE13_1x1_5.08V, J10 Conn_HE13_1x1_5.08V, J11 Conn_HE13_1x1_5.08V, J12 Conn_HE13_1x6_2.54H, J13 Conn_HE13_1x3_2.54V, J14 Conn_HE13_1x3_2.54V, J15 Conn_HE13_1x3_2.54V, J16 Conn_HE13_1x3_2.54V, J17 Conn_HE13_1x3_2.54V, J18 Conn_HE13_1x2_2.54V, J19 Conn_HE13_1x2_2.54V, J2 Conn_HE13_1x1_5.08V, J20 Conn_HE13_1x2_2.54V, J21 Conn_HE13_1x2_2.54V, J22 Conn_HE13_1x2_2.54V, J23 Conn_HE13_1x2_2.54V, J24 Conn_HE13_1x5_2.54V, J25 Conn_HE13_1x4_2.54V, J3 Conn_HE13_1x4_2.54V, J4 Conn_HE13_1x2_2.54V, J5 Conn_HE13_1x2_2.54V, J6 Conn_HE13_1x2_2.54V, J7 Conn_HE13_1x4_2.54V, J8 Conn_HE13_1x2_2.54V, J9 Conn_HE13_1x6_2.54H, M1 nRF24L01, U1 MAX487CSA_ESA

Commit message: wip
Parts:
- removed J3, J7: Conn_HE13_1x4_2.54V, p_Package_Misc:PinHeader_1x04_P2.54mm_Vertical, symbol p_Misc:Conn_HE13_1x4_2.54V
- removed J9: Conn_HE13_1x6_2.54H, p_Package_Misc:PinHeader_1x06_P2.54mm_Horizontal, symbol p_Misc:Conn_HE13_1x6_2.54H
- added H1, H2, H3, H4: drill_hole_5mm, p_Package_Misc:Drill_hole_5mm, symbol p_Misc:drill_hole_5mm
- added J10, J11, J12, J13, J7, J9: Conn_HE13_1x2_2.54V, p_Package_Misc:PinHeader_1x02_P2.54mm_Vertical, symbol p_Misc:Conn_HE13_1x2_2.54V
- added J3: Conn_HE13_1x6_2.54V, p_Package_Misc:PinHeader_1x06_P2.54mm_Vertical, symbol p_Misc:Conn_HE13_1x6_2.54V
- renumbered J10 to J14, J11 to J15, J12 to J16, J13 to J17, J14 to J18, J15 to J19, J16 to J20, J17 to J21, J18 to J22, J19 to J23, J20 to J24, J21 to J25, J22 to J26, J23 to J27, J24 to J28, J25 to J29
Connections:
- net input_stage/LOOPBACK1 is gone; now on net analog_input_stage/V_MONITOR2: J8.1
- net input_stage/LOOPBACK2 is gone; now on net GND: J8.2
- net +3.3V: now also J3.1
- net +BATT: now also R1.1; no longer R1.2
- net BAT_SENSE+: now also R1.4; no longer R1.3
- net BAT_SENSE-: now also R1.3; no longer R1.4
- net GND: now also H1.1 (H), H2.1 (H), H3.1 (H), H4.1 (H), J10.2, J11.2, J12.2, J13.2, J3.6, J7.2, J9.2
- net I2C_SCL: now also J3.3
- net I2C_SDA: now also J3.2
- net MCU/TEMP1: now also J4.1, R2.2; no longer J6.1, R5.2
- net MCU/TEMP3: now also J6.1, R5.2; no longer J4.1, R2.2
- net analog_input_stage/V_MONITOR1: now also J7.1
- net analog_input_stage/V_MONITOR3: now also J9.1
- net input_stage/INPUT1: now also J10.1
- net input_stage/INPUT2: now also J11.1
- net input_stage/INPUT3: now also J12.1
- net input_stage/INPUT4: now also J13.1
- net at J1.1: now also R1.2; no longer R1.1
- new net GPIO1: J3.4
- new net GPIO2: J3.5
Other:
- sheet MCU ports: added GPIO1, GPIO2; removed LOOPBACK1, LOOPBACK2
- sheet input_stage ports: added none; removed LOOPBACK1, LOOPBACK2, LP1, LP2
- note added: "Battery in / out"
- note added: "Input"
- note added: "Inter-board extension"
- note added: "Temperature sensors"
- note added: "Voltages monitoring"
- note removed: "Battery in / out connector"
- note removed: "I2C extension connector"
- note removed: "Input connector"
- note removed: "Loopback connector"
- note removed: "Temperature sensors connector"
- note removed: "Voltages monitoring connector"
- moved on the sheet: R1
