File: 02-hardware/wireless receiver/wireless receiver_first.kicad_pcb (KiCad board)
At the start: 2 copper layers, 58 x 78.7 mm, 123 parts, among them J1 Conn_HE13_1x1_5.08V, J10 Conn_HE13_1x2_2.54V, J11 Conn_HE13_1x2_2.54V, J12 Conn_HE13_1x2_2.54V, J13 Conn_HE13_1x2_2.54V, J14 Conn_HE13_1x1_5.08V, J15 Conn_HE13_1x1_5.08V, J16 Conn_HE13_1x6_2.54H, J17 Conn_HE13_1x3_2.54V, J18 Conn_HE13_1x3_2.54V, J19 Conn_HE13_1x3_2.54V, J2 Conn_HE13_1x1_5.08V, J20 Conn_HE13_1x3_2.54V, J21 Conn_HE13_1x3_2.54V, J22 Conn_HE13_1x2_2.54V, J23 Conn_HE13_1x2_2.54V, J24 Conn_HE13_1x2_2.54V, J25 Conn_HE13_1x2_2.54V, J26 Conn_HE13_1x2_2.54V, J27 Conn_HE13_1x2_2.54V, J28 Conn_HE13_1x5_2.54V, J29 Conn_HE13_1x4_2.54V, J3 Conn_HE13_1x6_2.54V, J4 Conn_HE13_1x2_2.54V, J5 Conn_HE13_1x2_2.54V, J6 Conn_HE13_1x2_2.54V, J7 Conn_HE13_1x2_2.54V, J8 Conn_HE13_1x2_2.54V, J9 Conn_HE13_1x2_2.54V, M1 nRF24L01, Q1 BC848B, Q2 BC848B, Q3 BC848B, Q4 BC848B, Q5 BC848B, U1 MAX487CSA_ESA, U10 STM32G030_C8, U11 74HCT244, U12 74HCT244, U2 TPS54332, U3 MCP1804T-5002I_O, U4 MCP1804T-3302I_O, U5 LMV824AIYDT, U6 MCP6N11-001E_SN, U7 74HCT244, U8 TCA9538, U9 REF193GSZ, Y1 Crystal_HC49CMS

Commit message: wip
Parts:
- moved C24 27.9 mm to (63.7, 117.1), turned to 135 degrees
- moved R28 25.3 mm to (76.1, 102.5), turned to -45 degrees
- moved C21 24.7 mm to (86.6, 123.4), turned to -135 degrees
- moved R29 23.4 mm to (75.0, 103.6), turned to -45 degrees
- moved C23 22.7 mm to (70.9, 124.3), turned to -45 degrees
- moved Y1 16.8 mm to (69.6, 118.1), turned to 135 degrees
- moved U9 15.6 mm to (83.6, 120.0), turned to 135 degrees
- moved J18 11.6 mm to (98.4, 93.2)
- moved R6 11.3 mm to (65.4, 100.8)
- moved D1 10.3 mm to (65.6, 103.3)
- moved U10 9.97 mm to (78.4, 110.2), turned to 45 degrees
- moved R27 9.91 mm to (72.6, 114.2), turned to 45 degrees
- moved R4 9.17 mm to (65.4, 99.3)
- moved C18 8.45 mm to (74.9, 118.5), turned to -45 degrees
- moved J19 7.68 mm to (98.4, 97.1)
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Connections:
- U10 pad 16: /MCU/ADC_CURRENT_MEAS -> /MCU/TEMP1
- U10 pad 24: /MCU/TEMP1 -> /MCU/ADC_CURRENT_MEAS
- U10 pad 37: /MCU/~{INT} -> /MCU/OUTPUT7
- U10 pad 41: /MCU/OUTPUT7 -> /MCU/~{INT}
- U11 pad 11: /MCU/OUTPUT1 -> /MCU/OUTPUT3
- U11 pad 12: /output_stage/OUTPUT2_LVL -> /output_stage/SERVO4_CMD
- U11 pad 13: /MCU/PWM4 -> /MCU/OUTPUT2
- U11 pad 15: /MCU/PWM5 -> /MCU/OUTPUT1
- U11 pad 16: /output_stage/OUTPUT3_LVL -> /output_stage/SERVO2_CMD
- U11 pad 17: /MCU/PWM2 -> /MCU/PWM5
- U11 pad 3: /output_stage/SERVO2_CMD -> /output_stage/SERVO5_CMD
- U11 pad 4: /MCU/OUTPUT3 -> /MCU/PWM2
- U11 pad 5: /output_stage/SERVO5_CMD -> /output_stage/OUTPUT1_LVL
- U11 pad 7: /output_stage/SERVO4_CMD -> /output_stage/OUTPUT2_LVL
- U11 pad 8: /MCU/OUTPUT2 -> /MCU/PWM4
- U11 pad 9: /output_stage/OUTPUT1_LVL -> /output_stage/OUTPUT3_LVL
Routing:
- net /MCU/OUTPUT4: track 60.7 -> 0.00 mm
- net /MCU/OUTPUT5: track 59.7 -> 0.00 mm
- net /MCU/OUTPUT6: track 58.9 -> 0.00 mm
- net /MCU/OUTPUT7: track 58.0 -> 0.00 mm
- net /SPI_MISO: track 0.03 -> 47.4 mm, vias 0 -> 1
- net /SWDIO: track 52.8 -> 8.65 mm, vias 1 -> 0
- net /SWCLK: track 50.3 -> 7.60 mm, vias 1 -> 0
- net /SPI_MOSI: track 8.56 -> 50.8 mm, vias 0 -> 1
- net /SPI_SCK: track 0.02 -> 40.0 mm, vias 0 -> 1
- net +5VP: track 5.17 -> 44.0 mm
- net /MCU/OUTPUT2: track 0.04 -> 33.3 mm, vias 0 -> 1
- net /MCU/~{INT}: track 28.5 -> 0.00 mm
- net /I2C_SDA: track 29.9 -> 2.41 mm, vias 1 -> 0
- net /MCU/INPUT3: track 27.4 -> 0.00 mm, vias 1 -> 0
- net /GPIO1: track 0.00 -> 26.4 mm, vias 0 -> 1
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